File: 2Cel_Bank.brd (EAGLE design)
At the start: 70 x 56 mm, 59 parts, among them IC1 CY8C4245-LQI-LONG, J1 DC-005, Q1 CSD17578Q3A, Q2 CSD17578Q3A, Q3 CSD17578Q3A, Q4 CSD17578Q3A, Q5 CSD25310Q2

Commit message: Route PCB
Parts:
- removed C1, C2, C3, C4, C5, C6: (no value), My_RLC:C0603
- removed DIS1: ER-OLED_BREACKOUT, Displays:ER-OLED_BRECKOUT
- removed F1: SMD1206R500SF, Seeed-OPL-fuse:F1812
- removed GG1: BQ28Z610, My_TI:VSON12
- removed IC1: CY8C4245-LQI-LONG, PsoC:QFN40-LONG
- removed JP1, JP2, JP3: (no value), pinhead:1X02
- removed POW1: 7805D2PAK, 74xx:D2PAK
- removed Q1, Q2: CSD17578Q3A, Mosfet_Logic:VSONP8
- removed R10, R4, R5, R6, R7, R9: (no value), My_RLC:R0603
- removed R21, R22, R8: (no value), rcl:R1206
- removed U$2: NSOT23, Mosfet_Logic:SOT23W
- added C13, C14, C18, C19, C20, C22: (no value), My_RLC:C0603
- added C15, C16, C17, C21: (no value), rcl:C0805
- added D1: (no value), diode:DO-214AC
- added DC/DC1: TPS61235, My_TI:VQFN9
- added DC/DC2: LM43603-Q1, My_TI:HTSSOP16PWP
- added L1, L2: 10UH, Seeed-OPL-Inductor:SMD-2P-L6.0XW6.0XH3.0MM
- added R27, R28: (no value), My_RLC:R0603
- R1, R2, R3: device My_RLC:R0603 -> rcl:R1206
- moved R1 47.4 mm to (3.00, 25.6), turned to 270 degrees
- moved R3 44.5 mm to (3.00, 30.4), turned to 90 degrees
- moved R2 36.6 mm to (67.8, 28.0)
- moved USB_CON1 23.4 mm to (50.4, 2.20)
- moved C11 5.39 mm to (51.0, 49.0), turned to 270 degrees
- moved R26 5.01 mm to (14.6, 8.60), turned to 180 degrees
- moved C10 2.99 mm to (54.8, 48.0), turned to 90 degrees
- moved Q5 2.00 mm to (10.6, 8.60)
- moved R25 1.80 mm to (14.6, 11.8)
- moved J1 1.60 mm to (18.8, 9.40)
- moved USB_CON2 0.40 mm to (20.0, 54.0)
Connections:
- net BAT2_PACK_MN renamed BAT_OUT_PACK_MN
- net BAT2_PACK_PL renamed BAT_OUT_PACK_PL
- removed net BAT1_PACK_MN: JP2.1, R22.2, R7.1, R8.1
- removed net BAT1_PACK_PL: C1.1, JP2.2, Q2.S1, Q2.S2, Q2.S3, R2.2, R21.2, R5.2, U$2.S
- removed net BAT1_PACK_SCL: GG1.5
- removed net BAT1_PACK_SDA: GG1.6
- removed net GND: POW1.GND
- removed net IN: POW1.IN
- removed net N$1: C2.2, F1.2, Q1.S1, Q1.S2, Q1.S3, R1.2
- removed net N$10: GG1.8, R5.1
- removed net N$12: GG1.11, R10.2
- removed net N$13: R6.1, U$2.G
- removed net N$14: C3.2, GG1.10
- removed net N$15: GG1.4, JP1.2
- removed net N$2: C4.1, C6.2, GG1.2, R7.2
- removed net N$27: GG2.4, JP3.2
- removed net N$3: Q1.D1, Q1.D2, Q1.D3, Q1.D4, Q1.D5, Q2.D1, Q2.D2, Q2.D3, Q2.D4, Q2.D5
- removed net N$4: Q2.G, R2.1, R3.2, U$2.D
- removed net N$5: Q1.G, R1.1, R4.2
- removed net N$6: C5.1, C6.1, GG1.3, R9.2
- removed net N$7: C1.2, C2.1
- removed net N$8: GG1.9, R4.1
- removed net N$9: GG1.7, R3.1
- removed net OUT: POW1.OUT
- removed net VCCA: IC1.33
- removed net VCCD: IC1.31
- new net BAT_PACK_MN: C10.2, C11.2, C9.1, GG2.1, GG2.EPAD_BIG, GG2.EPAD_M1, GG2.EPAD_M2, GG2.EPAD_M3, GG2.EPAD_M4, GG2.EPAD_VIA, R18.1, R19.2
- new net BAT_PACK_PL: F2.1, R20.1
- new net N$30: DC/DC1.1.1, DC/DC1.1.2, L1.2
- new net N$32: C13.2, DC/DC1.4
- new net N$33: C18.2, DC/DC2.1, DC/DC2.2, L2.2
- new net N$34: C15.1, C16.1, C17.1, DC/DC1.6, DC/DC1.9, USB_CON2.1
- new net N$35: C18.1, DC/DC2.3
- new net N$36: D1.A, USB_CON1.1
- new net N$37: C19.2, DC/DC2.4
- new net N$38: C22.2, DC/DC2.9, R27.2, R28.2
- net +24V: now also DC/DC2.12, DC/DC2.13, DC/DC2.14
- net BAT1_MN: now also R1.2; no longer C3.1, C4.2, C5.2, GG1.1, GG1.EPAD_BIG, GG1.EPAD_M1, GG1.EPAD_M2, GG1.EPAD_M3, GG1.EPAD_M4, GG1.EPAD_VIA, JP1.1, R8.2, R9.1
- net BAT1_PL: now also R2.1; no longer F1.1, R10.1
- net BAT2_MN: now also R3.2; no longer C10.2, C11.2, C9.1, GG2.1, GG2.EPAD_BIG, GG2.EPAD_M1, GG2.EPAD_M2, GG2.EPAD_M3, GG2.EPAD_M4, GG2.EPAD_VIA, JP3.1, R18.1, R19.2
- net BAT2_PL: now also R2.2; no longer F2.1, R20.1
- net PE: now also C13.1, C14.1, C15.2, C16.2, C17.2, C19.1, C20.1, C21.2, DC/DC1.1, DC/DC1.5, DC/DC1.8, DC/DC2.10, DC/DC2.15, DC/DC2.16, DC/DC2.6, DC/DC2.EXP, R1.1, R28.1, R3.1, USB_CON1.5, USB_CON2.5; no longer DIS1.GND, IC1.34, IC1.9, IC1.EPAD_B, IC1.EPAD_T, IC1.EPAD_VIA1, IC1.EPAD_VIA2, IC1.EPAD_VIA3, IC1.EPAD_VIA4, IC1.EPAD_VIA5, IC1.EPAD_VIA6, IC1.EPAD_VIA7, IC1.EPAD_VIA8, IC1.EPAD_VIA9, R22.1, R6.2, USB_CON1.P$1, USB_CON1.P$2, USB_CON1.P$3, USB_CON1.P$4, USB_CON2.P$1, USB_CON2.P$2, USB_CON2.P$3, USB_CON2.P$4
- net VCC: now also C14.2, C20.2, C21.1, C22.1, D1.C, DC/DC1.3, DC/DC1.7, DC/DC2.5, L1.1, L2.1, R27.1; no longer IC1.32, R21.1
Routing:
- net +24V: track 4.41 -> 48.1 mm, vias 0 -> 1
- net BAT1_PACK_PL: track 33.7 -> 0.00 mm, vias 2 -> 0
- net N$27: track 32.7 -> 0.00 mm, vias 1 -> 0
- net VCC: track 38.8 -> 63.6 mm
- net N$15: track 23.9 -> 0.00 mm, vias 1 -> 0
- net N$34: track 0.00 -> 22.1 mm
- net BAT_OUT_PACK_PL: track 32.9 -> 53.6 mm
- net BAT1_PL: track 20.1 -> 0.00 mm
- net N$4: track 19.8 -> 0.00 mm
- net BAT2_PL: track 20.7 -> 4.00 mm
- net N$33: track 0.00 -> 14.4 mm
- net N$6: track 12.6 -> 0.00 mm, vias 2 -> 0
- net BAT1_PACK_MN: track 12.6 -> 0.00 mm
- net N$30: track 0.00 -> 12.2 mm, vias 0 -> 2
- net N$2: track 11.7 -> 0.00 mm
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- added copper zone on layer 1, net BAT_PACK_MN
- added copper zone on layer 16, net BAT_PACK_MN
- added copper zone on layer 1, net PE
- removed copper zone on layer 1, net BAT1_MN
- removed copper zone on layer 16, net BAT1_MN
- removed copper zone on layer 16, net BAT1_PACK_PL
- removed copper zone on layer 1, net BAT2_MN
- removed copper zone on layer 16, net BAT2_MN
- removed copper zone on layer 16, net BAT_OUT_PACK_PL

Commit message: Complite Route
Parts:
- removed C15: (no value), rcl:C0805
- removed USB_CON2: MICRO_USB_2.0, Interface:MICRO-USB5+4P-SMD-0.65
- added C1, C2, C23, C24, C25, C26, C27, C28, C29, C3, C30, C31, C32, C33, C34, C35, C4, C5, C6: (no value), My_RLC:C0603
- added C36, C37, C38, C39: (no value), rcl:SMC_A
- added C40: (no value), rcl:SMC_D
- added CH1: BQ25070, My_TI:DFN10_2X3
- added DC/DC3: TPS63030, My_TI:WSON10
- added IC1: (no value), Interface:QFN-28
- added JP1: (no value), pinhead:1X05
- added L3: (no value), My_RLC:L0603
- added LED1, LED2, LED4: (no value), led:CHIP-LED0603
- added R10, R21, R22, R29, R30, R31, R32, R33, R4, R5, R6, R7, R8, R9: (no value), My_RLC:R0603
- added U$1: CY8C4245, PsoC:TQFP44_CY_LOGO
- added U$2: 5032ACTIVE, Oscillatrs:5030A
- added U$4: ER-OLED_0.96, Displays:30PIN
- added U$5: NSOT23, Mosfet_Logic:SOT23W
- added X1: (no value), con-usb-3:USB-A-S
- moved DC/DC1 8.35 mm to (34.4, 52.4)
- moved C13 7.96 mm to (36.8, 54.8), turned to 270 degrees
- moved C14 6.32 mm to (37.6, 52.2), turned to 180 degrees
- moved C16 5.66 mm to (30.0, 47.2), turned to 270 degrees
- moved C17 5.10 mm to (23.4, 47.4), turned to 180 degrees
Connections:
- removed net BAT2_PACK_SCL: GG2.5
- removed net BAT2_PACK_SDA: GG2.6
- new net DISPLAY_RESET: U$1.38, U$4.14
- new net N$1: C1.2, IC1.18
- new net N$10: C24.2, U$4.5
- new net N$12: C28.1, U$4.27
- new net N$13: R6.2, U$4.26
- new net N$14: R10.1, R21.1, U$1.4
- new net N$15: C27.1, U$4.28
- new net N$2: IC1.9, R4.2
- new net N$27: R7.1, U$4.11
- new net N$3: JP1.5, U$1.13
- new net N$39: DC/DC3.P$4, L3.1
- new net N$4: JP1.4, U$1.14
- new net N$40: C29.1, DC/DC3.P$6, DC/DC3.P$7, DC/DC3.P$8
- new net N$41: CH1.P$1, D1.C
- new net N$42: CH1.P$2, R22.2
- new net N$43: LED1.C, U$5.S
- new net N$44: CH1.P$5, R29.2, R30.1
- new net N$46: LED1.A, R31.2
- new net N$47: R33.1, U$1.5
- new net N$48: LED2.A, R32.2
- new net N$49: LED4.A, R33.2
- new net N$5: C5.2, U$1.33
- new net N$50: R32.1, U$1.6
- new net N$6: R5.2, U$2.1
- new net N$7: C23.1, U$4.2
- new net N$8: C24.1, U$4.4
- new net N$9: C23.2, U$4.3
- new net PSOC_RESET: JP1.3, U$1.32
- new net SCL: GG2.5, R8.2, U$1.28, U$4.18
- new net SCLK: U$1.30, U$2.3
- new net SDA: GG2.6, R9.2, U$1.29, U$4.19, U$4.20
- new net USB_CHARGE_CONTROLL: CH1.P$7, U$1.25
- new net USB_CHARGE_STATUS: CH1.P$8, U$1.24
- new net USB_D+: IC1.4, USB_CON1.3
- new net USB_D-: IC1.5, USB_CON1.2
- new net USB_DETECT: C33.2, CH1.P$4, R30.2
- new net USB_RX: IC1.25, U$1.21
- new net USB_TX: IC1.26, U$1.20
- new net VBUS: C2.1, C3.1, D1.A, IC1.7, IC1.8, R4.1, USB_CON1.1
- new net VDD: C25.2, C26.1, C31.1, C32.1, C34.1, C35.1, C36.+, C37.+, C4.1, C6.1, DC/DC3.P$1, DC/DC3.P$10, IC1.6, JP1.1, R5.1, R7.2, R8.1, R9.1, U$1.19, U$1.34, U$1.35, U$2.4, U$4.6, U$4.9
- new net WAKEUP: U$1.31
- net +24V: now also C40.+
- net BAT1_PL: now also R10.2
- net BAT_OUT_PACK_PL: now also C30.2, CH1.P$10, CH1.P$6, DC/DC3.P$5
- net N$31: now also U$5.G
- net N$34: now also C39.+, X1.VBUS; no longer C15.1, USB_CON2.1
- net N$36: now also DC/DC3.P$2, L3.2; no longer D1.A, USB_CON1.1
- net PE: now also C1.1, C2.2, C25.1, C26.2, C27.2, C28.2, C29.2, C3.2, C30.1, C31.2, C32.2, C33.1, C34.2, C35.2, C36.-, C37.-, C38.-, C39.-, C4.2, C40.-, C5.1, C6.2, CH1.EPAD, CH1.P$3, CH1.P$9, DC/DC3.EPAD_B, DC/DC3.EPAD_T, DC/DC3.EPAD_VIA, DC/DC3.P$3, DC/DC3.P$9, IC1.3, IC1.EPAD_B, IC1.EPAD_T, IC1.EPAD_VIA1, IC1.EPAD_VIA2, IC1.EPAD_VIA3, IC1.EPAD_VIA4, IC1.EPAD_VIA5, IC1.EPAD_VIA6, IC1.EPAD_VIA7, IC1.EPAD_VIA8, IC1.EPAD_VIA9, JP1.2, LED2.C, LED4.C, R21.2, R22.1, R29.1, R6.1, U$1.1, U$1.10, U$1.36, U$2.2, U$4.10, U$4.12, U$4.13, U$4.15, U$4.16, U$4.17, U$4.21, U$4.22, U$4.23, U$4.24, U$4.25, U$4.29, U$4.30, U$4.8, U$5.D, X1.GND; no longer C15.2, USB_CON2.5
- net VCC: now also C38.+, R31.1; no longer D1.C
Routing:
- net VDD: track 0.00 -> 122.8 mm, vias 0 -> 3
- net SDA: track 0.00 -> 67.4 mm, vias 0 -> 3
- net SCL: track 0.00 -> 66.3 mm, vias 0 -> 3
- net VCC: track 63.6 -> 118.6 mm, vias 2 -> 4
- net N$14: track 0.00 -> 47.2 mm, vias 0 -> 2
- net BAT_OUT_PACK_PL: track 53.6 -> 91.5 mm, vias 2 -> 4
- net VBUS: track 0.00 -> 33.5 mm, vias 0 -> 2
- net PE: track 23.5 -> 54.6 mm, vias 6 -> 10
- net PSOC_RESET: track 0.00 -> 23.9 mm, vias 0 -> 1
- net N$41: track 0.00 -> 22.3 mm, vias 0 -> 2
- net N$4: track 0.00 -> 20.6 mm
- net N$3: track 0.00 -> 20.5 mm
- net DISPLAY_RESET: track 0.00 -> 17.9 mm, vias 0 -> 2
- net BAT2_MN: track 2.18 -> 18.0 mm
- net BAT1_MN: track 2.18 -> 17.2 mm
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Other:
- board text added: "1"
- board text added: "30"
