File: 2Cel_Bank.sch (EAGLE design)
At the start: 59 parts, among them IC1 CY8C4245-LQI-LONG, J1 DC-005, Q1 CSD17578Q3A, Q2 CSD17578Q3A, Q3 CSD17578Q3A, Q4 CSD17578Q3A, Q5 CSD25310Q2

Commit message: Route PCB
Parts:
- removed C1, C2, C3, C4, C5, C6: (no value), My_RLC:CAP0603
- removed DIS1: ER-OLED_BREACKOUT, Displays:ER-OLED_BREACKOUT
- removed F1: SMD1206R500SF, Seeed-OPL-fuse:SMD-PPTC-500MA-15V(1812)
- removed GG1: BQ28Z610, My_TI:BQ28Z610
- removed IC1: CY8C4245-LQI-LONG, PsoC:CY8C4245-LQI-LONG
- removed JP1, JP2, JP3: (no value), pinhead:PINHD-1X2
- removed POW1: 7805D2PAK, 74xx:7805D2PAK
- removed Q1, Q2: CSD17578Q3A, Mosfet_Logic:CSD17578Q3A
- removed R10, R4, R5, R6, R7, R9: (no value), My_RLC:RES0603
- removed R21, R22, R8: (no value), rcl:R-EU_R1206
- removed U$2: NSOT23, Mosfet_Logic:NSOT23
- added C13, C14, C18, C19, C20, C22: (no value), My_RLC:CAP0603
- added C15, C16, C17, C21: (no value), rcl:C-EUC0805
- added D1: (no value), diode:DIODE-DO-214AC
- added DC/DC1: TPS61235, My_TI:TPS61235
- added DC/DC2: LM43603-Q1, My_TI:LM43603-Q1
- added L1, L2: 10UH, Seeed-OPL-Inductor:SMD-INDUCTOR-10UH-20%(2P-6X6MM)'0630'
- added R27, R28: (no value), My_RLC:RES0603
- R1, R2, R3: device My_RLC:RES0603 -> rcl:R-EU_R1206
Connections:
- net BAT2_PACK_MN renamed BAT_OUT_PACK_MN
- net BAT2_PACK_PL renamed BAT_OUT_PACK_PL
- removed net BAT1_PACK_MN: JP2.1, R22.2, R7.P$1, R8.1
- removed net BAT1_PACK_PL: C1.P$1, JP2.2, Q2.S, R2.P$2, R21.2, R5.P$2, U$2.S
- removed net BAT1_PACK_SCL: GG1.P$5
- removed net BAT1_PACK_SDA: GG1.P$6
- removed net N$1: C2.P$2, F1.2, Q1.S, R1.P$2
- removed net N$10: GG1.P$8, R5.P$1
- removed net N$12: GG1.P$11, R10.P$2
- removed net N$13: R6.P$1, U$2.G
- removed net N$14: C3.P$2, GG1.P$10
- removed net N$15: GG1.P$4, JP1.2
- removed net N$2: C4.P$1, C6.P$2, GG1.P$2, R7.P$2
- removed net N$27: GG2.P$4, JP3.2
- removed net N$3: Q1.D, Q2.D
- removed net N$4: Q2.G, R2.P$1, R3.P$2, U$2.D
- removed net N$5: Q1.G, R1.P$1, R4.P$2
- removed net N$6: C5.P$1, C6.P$1, GG1.P$3, R9.P$2
- removed net N$7: C1.P$2, C2.P$1
- removed net N$8: GG1.P$9, R4.P$1
- removed net N$9: GG1.P$7, R3.P$1
- new net BAT_PACK_MN: C10.P$2, C11.P$2, C9.P$1, GG2.P$1, GG2.P$13, R18.P$1, R19.2
- new net BAT_PACK_PL: F2.1, R20.P$1
- new net N$30: DC/DC1.P$2, L1.2
- new net N$32: C13.P$2, DC/DC1.P$4
- new net N$33: C18.P$2, DC/DC2.P$1, DC/DC2.P$2, L2.2
- new net N$34: C15.1, C16.1, C17.1, DC/DC1.P$6, DC/DC1.P$9, USB_CON2.P$1
- new net N$35: C18.P$1, DC/DC2.P$3
- new net N$36: D1.A, USB_CON1.P$1
- new net N$37: C19.P$2, DC/DC2.P$4
- new net N$38: C22.P$2, DC/DC2.P$9, R27.P$2, R28.P$2
- net +24V: now also DC/DC2.P$12, DC/DC2.P$13, DC/DC2.P$14
- net BAT1_MN: now also R1.2; no longer C3.P$1, C4.P$2, C5.P$2, GG1.P$1, GG1.P$13, JP1.1, R8.2, R9.P$1
- net BAT1_PL: now also R2.1; no longer F1.1, R10.P$1
- net BAT2_MN: now also R3.2; no longer C10.P$2, C11.P$2, C9.P$1, GG2.P$1, GG2.P$13, JP3.1, R18.P$1, R19.2
- net BAT2_PL: now also R2.2; no longer F2.1, R20.P$1
- net PE: now also C13.P$1, C14.P$1, C15.2, C16.2, C17.2, C19.P$1, C20.P$1, C21.2, DC/DC1.P$1, DC/DC1.P$5, DC/DC1.P$8, DC/DC2.P$10, DC/DC2.P$15, DC/DC2.P$16, DC/DC2.P$6, R1.1, R28.P$1, R3.1, USB_CON1.P$5, USB_CON2.P$5; no longer DIS1.GND, IC1.GND, IC1.GNDA, R22.1, R6.P$2, USB_CON1.P$6, USB_CON2.P$6
- net VCC: now also C14.P$2, C20.P$2, C21.1, C22.P$1, D1.C, DC/DC1.P$3, DC/DC1.P$7, DC/DC2.P$5, L1.1, L2.1, R27.P$1; no longer R21.1
Other:
- moved on the sheet: F2, GG2, JP4, Q3, Q4, R19, R23, R24, U$3

Commit message: Complite Route
Parts:
- removed C15: (no value), rcl:C-EUC0805
- removed USB_CON2: MICRO_USB_2.0, Interface:MICRO_USB_2.0
- added C1, C2, C23, C24, C25, C26, C27, C28, C29, C3, C30, C31, C32, C33, C34, C35, C4, C5, C6: (no value), My_RLC:CAP0603
- added C36, C37, C38, C39: (no value), rcl:CPOL-EUSMCA
- added C40: (no value), rcl:CPOL-EUSMCD
- added CH1: BQ25070, My_TI:BQ25070
- added DC/DC3: TPS63030, My_TI:TPS63030
- added IC1: (no value), Interface:CP2102/9
- added JP1: (no value), pinhead:PINHD-1X5
- added L3: (no value), My_RLC:L0603
- added LED1, LED2, LED4: (no value), led:LEDCHIP-LED0603
- added R10, R21, R22, R29, R30, R31, R32, R33, R4, R5, R6, R7, R8, R9: (no value), My_RLC:RES0603
- added U$1: CY8C4245, PsoC:CY8C4245
- added U$2: 5032ACTIVE, Oscillatrs:5032ACTIVE
- added U$4: ER-OLED_0.96, Displays:ER-OLED_0.96
- added U$5: NSOT23, Mosfet_Logic:NSOT23
- added X1: (no value), con-usb-3:USB-A-S
Connections:
- removed net BAT2_PACK_SCL: GG2.P$5
- removed net BAT2_PACK_SDA: GG2.P$6
- new net DISPLAY_RESET: U$1.38, U$4.14
- new net N$1: C1.P$2, IC1.P$18
- new net N$10: C24.P$2, U$4.5
- new net N$12: C28.P$1, U$4.27
- new net N$13: R6.P$2, U$4.26
- new net N$14: R10.P$1, R21.P$1, U$1.4
- new net N$15: C27.P$1, U$4.28
- new net N$2: IC1.P$9, R4.P$2
- new net N$27: R7.P$1, U$4.11
- new net N$3: JP1.5, U$1.13
- new net N$39: DC/DC3.P$4, L3.P$1
- new net N$4: JP1.4, U$1.14
- new net N$40: C29.P$1, DC/DC3.P$6, DC/DC3.P$7, DC/DC3.P$8
- new net N$41: CH1.P$1, D1.C
- new net N$42: CH1.P$2, R22.P$2
- new net N$43: LED1.C, U$5.S
- new net N$44: CH1.P$5, R29.P$2, R30.P$1
- new net N$46: LED1.A, R31.P$2
- new net N$47: R33.P$1, U$1.5
- new net N$48: LED2.A, R32.P$2
- new net N$49: LED4.A, R33.P$2
- new net N$5: C5.P$2, U$1.33
- new net N$50: R32.P$1, U$1.6
- new net N$6: R5.P$2, U$2.EN
- new net N$7: C23.P$1, U$4.2
- new net N$8: C24.P$1, U$4.4
- new net N$9: C23.P$2, U$4.3
- new net PSOC_RESET: JP1.3, U$1.32
- new net SCL: GG2.P$5, R8.P$2, U$1.28, U$4.18
- new net SCLK: U$1.30, U$2.OUT
- new net SDA: GG2.P$6, R9.P$2, U$1.29, U$4.19, U$4.20
- new net USB_CHARGE_CONTROLL: CH1.P$7, U$1.25
- new net USB_CHARGE_STATUS: CH1.P$8, U$1.24
- new net USB_D+: IC1.P$4, USB_CON1.P$3
- new net USB_D-: IC1.P$5, USB_CON1.P$2
- new net USB_DETECT: C33.P$2, CH1.P$4, R30.P$2
- new net USB_RX: IC1.P$25, U$1.21
- new net USB_TX: IC1.P$26, U$1.20
- new net VBUS: C2.P$1, C3.P$1, D1.A, IC1.P$7, IC1.P$8, R4.P$1, USB_CON1.P$1
- new net VDD: C25.P$2, C26.P$1, C31.P$1, C32.P$1, C34.P$1, C35.P$1, C36.+, C37.+, C4.P$1, C6.P$1, DC/DC3.P$1, DC/DC3.P$10, IC1.P$6, JP1.1, R5.P$1, R7.P$2, R8.P$1, R9.P$1, U$1.19, U$1.34, U$1.35, U$2.+5V, U$4.6, U$4.9
- new net WAKEUP: U$1.31
- net +24V: now also C40.+
- net BAT1_PL: now also R10.P$2
- net BAT_OUT_PACK_PL: now also C30.P$2, CH1.P$10, CH1.P$6, DC/DC3.P$5
- net N$31: now also U$5.G
- net N$34: now also C39.+, X1.VBUS; no longer C15.1, USB_CON2.P$1
- net N$36: now also DC/DC3.P$2, L3.P$2; no longer D1.A, USB_CON1.P$1
- net PE: now also C1.P$1, C2.P$2, C25.P$1, C26.P$2, C27.P$2, C28.P$2, C29.P$2, C3.P$2, C30.P$1, C31.P$2, C32.P$2, C33.P$1, C34.P$2, C35.P$2, C36.-, C37.-, C38.-, C39.-, C4.P$2, C40.-, C5.P$1, C6.P$2, CH1.P$3, CH1.P$9, DC/DC3.P$3, DC/DC3.P$9, IC1.P$3, JP1.2, LED2.C, LED4.C, R21.P$2, R22.P$1, R29.P$1, R6.P$1, U$1.1, U$1.10, U$1.36, U$2.GND, U$4.10, U$4.12, U$4.13, U$4.15, U$4.16, U$4.17, U$4.21, U$4.22, U$4.23, U$4.24, U$4.25, U$4.29, U$4.30, U$4.8, U$5.D, X1.GND; no longer C15.2, USB_CON2.P$5
- net VCC: now also C38.+, R31.P$1; no longer D1.C
